Commit message: test jump

File: robots/atlas/urdf/atlas_legs_only.urdf (robot description, URDF)
Before this commit: robot atlas, 16 links, 15 joints
Joints:
- joint back_bkx: limit lower=-0.523599 upper=0.523599 effort=300 velocity=12 -> lower=-0.523599 upper=0.523599 effort=300 velocity=1
- joint back_bky: limit lower=-0.219388 upper=0.538783 effort=445 velocity=9 -> lower=-0.219388 upper=0.538783 effort=445 velocity=12
- joint back_bkz: limit lower=-0.663225 upper=0.663225 effort=106 velocity=12 -> lower=-0.663225 upper=0.663225 effort=106 velocity=1
