Commit message: edit joint name

File: robots/singleleg/singleleg.urdf (robot description, URDF)
Before this commit: robot singleleg, 4 links, 3 joints
Joints:
- removed joint joint_low_leg
- removed joint joint_up_leg
- added joint joint_hip: type revolute, parent pelvis, child up_leg, origin xyz=0 0 -0.03 rpy=0 0 0, axis 0 -1 0, limit lower=-3.14 upper=3.14 effort=100 velocity=1
- added joint joint_knee: type revolute, parent up_leg, child low_leg, origin xyz=0 0 -0.05 rpy=0 0 0, axis 0 -1 0, limit lower=-3.14 upper=3.14 effort=100 velocity=1

Commit message: add singlelegmultibody

File: robots/singleleg/singleleg.urdf (robot description, URDF)
Before this commit: robot singleleg, 4 links, 3 joints
Links:
- removed link pelvis
- added link body, mass 7.9; collision mesh filename=meshes/body.obj; visual mesh filename=meshes/body.obj
Joints:
- joint joint_hip: parent pelvis -> body

Commit message: replace urdf; add singlelegjump

File: robots/singleleg/singleleg.urdf (robot description, URDF)
Before this commit: robot singleleg, 4 links, 3 joints
Links:
- link body: mass 7.9 -> 4; geometry collision mesh filename=meshes/body.STL; visual mesh filename=meshes/body.STL
- link heel: mass 0.1 -> 2; geometry collision mesh filename=meshes/heel.STL; visual mesh filename=meshes/heel.STL
- link low_leg: mass 1 -> 2; geometry collision mesh filename=meshes/low_leg.STL; visual mesh filename=meshes/low_leg.STL
- link up_leg: mass 1 -> 2; geometry collision mesh filename=meshes/up_leg.STL; visual mesh filename=meshes/up_leg.STL
Joints:
- removed joint joint_ankle
- removed joint joint_hip
- removed joint joint_knee
- added joint joint_hell: type revolute, parent low_leg, child heel, origin xyz=-0.00532262680792502 0 -0.05 rpy=0 0 0, axis 0 1 0, limit lower=-3.14 upper=3.14 effort=100 velocity=1
- added joint joint_low_leg: type revolute, parent up_leg, child low_leg, origin xyz=0 0 -0.05 rpy=0 0 0, axis 0 -1 0, limit lower=-3.14 upper=3.14 effort=100 velocity=1
- added joint joint_up_leg: type revolute, parent body, child up_leg, origin xyz=0 0 -0.03 rpy=0 0 0, axis 0 -1 0, limit lower=-3.14 upper=3.14 effort=100 velocity=1

File: robots/singleleg/singlelegtwocontact.urdf (robot description, URDF)
Before this commit: robot singleleg, 4 links, 3 joints
Joints:
- joint joint_ankle: origin xyz=0 0 -0.0525 rpy=0 0 0 -> xyz=-0.00532262680792502 0 -0.05 rpy=0 0 0
